File: kicad/shaun-proj/shaun-proj.kicad_pcb (KiCad board)
At the start: 2 copper layers, 57 parts, among them J1 USB_C_Receptacle_USB2.0_16P, J2 Conn_02x16_Odd_Even, J3 Conn_01x02_Socket, Q1 AO3401A, Q2 AO3400A, Q3 AO3401A, Q4 AO3400A, Q5 AO3400A, Q6 AO3401A, SW2 SW_SPDT, U1 CH224K, U2 TPS5430DDA, U3 INA219AxD, U5 TP4056-42-ESOP8

Commit message: major improvements, components layout + pcb, parts, tests, i2c stuff, ++
Parts:
- added JP3: SolderJumper_2_Open, Jumper:SolderJumper-2_P1.3mm_Open_TrianglePad1.0x1.5mm, F.Cu at (124.5, 65.5)
- added JP4: SolderJumper_2_Open, Jumper:SolderJumper-2_P1.3mm_Open_TrianglePad1.0x1.5mm, F.Cu at (133.5, 78.8)
- added JP5: SolderJumper_2_Open, Jumper:SolderJumper-2_P1.3mm_Open_TrianglePad1.0x1.5mm, F.Cu at (133.5, 82.2)
- added R19: 100m, Resistor_SMD:R_1206_3216Metric_Pad1.30x1.75mm_HandSolder, F.Cu at (126.5, 76.3)
- added R2: 10k, Resistor_SMD:R_0603_1608Metric_Pad0.98x0.95mm_HandSolder, F.Cu at (123.0, 57.0)
- added R20: 3.3k, Resistor_SMD:R_0603_1608Metric_Pad0.98x0.95mm_HandSolder, F.Cu at (128.9, 88.5)
- added R21: 3.3k, Resistor_SMD:R_0603_1608Metric_Pad0.98x0.95mm_HandSolder, F.Cu at (131.0, 90.5)
- D2: value LED -> GREEN LED
- JP1, JP2: value Jumper_2_Open -> SolderJumper_2_Open; footprint TestPoint:TestPoint_2Pads_Pitch2.54mm_Drill0.8mm -> Jumper:SolderJumper-2_P1.3mm_Open_TrianglePad1.0x1.5mm
- R9: value 50m -> 100m; footprint Resistor_SMD:R_1206_3216Metric -> Resistor_SMD:R_1206_3216Metric_Pad1.30x1.75mm_HandSolder
- moved TP11 66.8 mm to (135.0, 86.5)
- moved TP4 63.9 mm to (114.0, 66.5)
- moved TP9 61.8 mm to (122.5, 73.0)
- moved TP13 60.8 mm to (127.5, 70.0)
- moved TP1 60.1 mm to (120.0, 64.0)
- moved TP5 55.2 mm to (119.5, 55.5)
- moved TP8 49.1 mm to (139.5, 72.5)
- moved TP7 47.4 mm to (133.5, 55.0)
- moved TP2 47.3 mm to (132.5, 64.0)
- moved TP10 41.3 mm to (137.0, 55.0)
- moved TP14 35.0 mm to (155.5, 69.0)
- moved JP2 32.3 mm to (132.0, 87.5), turned to -90 degrees
- moved R9 21.9 mm to (126.5, 74.0), turned to 0 degrees
- moved JP1 21.7 mm to (126.0, 87.5), turned to -90 degrees
- moved Q5 21.3 mm to (175.6, 82.6)
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Connections:
- JP1 pad 1: VBUS -> I2C1_SDA
- JP1 pad 2: HV -> Net-(JP1-B)
- JP2 pad 1: BATTERY_POWER -> I2C1_SCL
- JP2 pad 2: 3V3_OUT -> Net-(JP2-B)
- R12 pad 2: Net-(U3-A1) -> Net-(U3-A0)
- U1 pad 8: VBUS -> Net-(U1-VBUS)
- U3 pad 1: Net-(U3-A1) -> GND
- U3 pad 2: GND -> Net-(U3-A0)
- U3 pad 5: 3V3_OUT -> Net-(JP4-A)
Other:
- board text added: "JLCJLCJLCJLC"
