File: kicad/shaun-proj/shaun-proj.kicad_pcb (KiCad board)
At the start: 2 copper layers, 94 parts, among them J1 USB_C_Receptacle_USB2.0_16P, J2 Conn_02x16_Odd_Even, J3 Conn_01x02_Socket, Q1 AO3401A, Q2 AO3400A, Q3 AO3401A, Q4 AO3400A, Q5 AO3400A, Q6 AO3401A, SW2 SW_SPDT, U1 CH224K, U2 TPS5430DDA, U3 INA219AxD, U4 DRV8833PWPR, U5 TP4056-42-ESOP8, U6 TPS63020DSJR, U7 DRV8833PWPR, U8 TPS63020DSJR

Commit message: da board
Parts:
- removed C7: 100n, Capacitor_SMD:C_0603_1608Metric_Pad1.08x0.95mm_HandSolder
- removed TP13, TP4, TP5, TP9: TestPoint, TestPoint:TestPoint_Pad_D1.5mm
- added G***: LOGO, MyLibrary:UCT_LOGO, F.Cu at (152.0, 68.2)
- added G***: LOGO, MyLibrary:Olympia, B.Cu at (148.5, 49.5)
- added G***: LOGO, MyLibrary:PommeDarker, B.Cu at (146.8, 99.2)
- added H1: MountingHole, MountingHole:MountingHole_3.2mm_M3, F.Cu at (141.0, 75.0)
- added R28: 100m, Resistor_SMD:R_1206_3216Metric_Pad1.30x1.75mm_HandSolder, F.Cu at (176.0, 54.2)
- added R29: 1, Resistor_SMD:R_0805_2012Metric_Pad1.20x1.40mm_HandSolder, F.Cu at (176.2, 62.5)
- added R35: 100m, Resistor_SMD:R_1206_3216Metric_Pad1.30x1.75mm_HandSolder, F.Cu at (173.8, 50.5)
- added R36: 1, Resistor_SMD:R_0805_2012Metric_Pad1.20x1.40mm_HandSolder, F.Cu at (155.0, 92.5)
- added REF**: OSHW-Logo2_7.3x6mm_SilkScreen, Symbol:OSHW-Logo2_7.3x6mm_SilkScreen, F.Cu at (151.5, 74.0)
- added REF**: KiCad-Logo2_5mm_SilkScreen, Symbol:KiCad-Logo2_5mm_SilkScreen, F.Cu at (146.2, 71.5)
- L4, L5, L6: footprint Inductor_SMD:L_Murata_DFE201610P -> Inductor_SMD:L_1008_2520Metric_Pad1.43x2.20mm_HandSolder
- R10, R6: value 1M -> 10k
- R4: value 560 -> 2k
- U1: footprint Package_SO:SSOP-10-1EP_3.9x4.9mm_P1mm_EP2.1x3.3mm -> Package_SO:SSOP-10-1EP_3.9x4.9mm_P1mm_EP2.1x3.3mm_ThermalVias
- U4, U7: footprint Package_SO:HTSSOP-16-1EP_4.4x5mm_P0.65mm_EP3x3mm -> Package_SO:HTSSOP-16-1EP_4.4x5mm_P0.65mm_EP3.4x5mm_Mask2.46x2.31mm_ThermalVias
- U5: footprint Package_SO:SOIC-8-1EP_3.9x4.9mm_P1.27mm_EP2.41x3.3mm -> Package_SO:SOIC-8-1EP_3.9x4.9mm_P1.27mm_EP2.41x3.3mm_ThermalVias
- U6, U8: footprint Package_SON:Texas_S-PWSON-N10_ThermalVias -> MyLibrary:DAMOLA_VSON-14-1EP_3.4x4.4mm_P0.5mm_EP1.6x4.2mm
- moved R23 76.8 mm to (137.1, 91.8), turned to 90 degrees
- moved L5 75.0 mm to (136.9, 96.0), turned to -90 degrees
- moved R24 73.6 mm to (138.3, 88.9)
- moved C14 73.1 mm to (143.9, 89.8), turned to 90 degrees
- moved L4 72.7 mm to (140.6, 96.8)
- moved R25 69.9 mm to (142.1, 88.3), turned to -90 degrees
- moved SW2 66.7 mm to (169.3, 104.8), turned to 0 degrees
- moved C15 63.8 mm to (143.9, 93.5), turned to 90 degrees
- moved L6 62.0 mm to (152.1, 54.8), turned to 180 degrees
- moved U6 61.1 mm to (140.6, 92.5), turned to 90 degrees
- moved C13 57.0 mm to (139.8, 82.5), turned to 180 degrees
- moved R34 56.3 mm to (151.6, 63.4), turned to 90 degrees
- moved R33 55.9 mm to (155.0, 94.5), turned to 180 degrees
- moved C22 54.8 mm to (153.3, 63.2), turned to -90 degrees
- moved J1 54.2 mm to (164.5, 42.0), turned to 90 degrees
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Connections:
- C14 pad 1: /Damola's Sheet/CONN1 -> Net-(U6-EN)
- C22 pad 1: /Damola's Sheet/CONN2 -> Net-(U8-EN)
- C5 pad 1: BATTERY -> CHARGE_BATTERY
- J2 pad 1: MOTOR2_B_OUT -> MOTOR2_A_OUT
- J2 pad 10: MOTOR4_CTRL2 -> unconnected-(J2-Pin_10-Pad10)
- J2 pad 11: EXT_LOAD2_OUT -> unconnected-(J2-Pin_11-Pad11)
- J2 pad 12: unconnected-(J2-Pin_12-Pad12) -> EXT_LOAD2_OUT
- J2 pad 13: FAST_CHARGE_CTRL -> BATTERY
- J2 pad 14: BATTERY -> FAST_CHARGE_CTRL
- J2 pad 15: unconnected-(J2-Pin_15-Pad15) -> I2C1_SCL
- J2 pad 16: I2C1_SCL -> unconnected-(J2-Pin_16-Pad16)
- J2 pad 17: I2C1_SDA -> 3V3_OUT
- J2 pad 18: 3V3_OUT -> I2C1_SDA
- J2 pad 19: GND -> 5V_OUT
- J2 pad 2: MOTOR2_A_OUT -> MOTOR2_B_OUT
- J2 pad 20: 5V_OUT -> GND
- J2 pad 21: EXT_LOAD1_OUT -> HV
- J2 pad 22: HV -> EXT_LOAD1_OUT
- J2 pad 23: GND -> MOTOR3_CTRL1
- J2 pad 24: MOTOR3_CTRL1 -> GND
- J2 pad 25: CTRL_EXT_LOAD1 -> MOTOR3_CTRL2
- J2 pad 26: MOTOR3_CTRL2 -> CTRL_EXT_LOAD1
- J2 pad 27: MOTOR3_A_OUT -> MOTOR1_CTRL1
- J2 pad 28: MOTOR1_CTRL1 -> MOTOR3_A_OUT
- J2 pad 29: MOTOR3_B_OUT -> MOTOR1_CTRL2
- J2 pad 3: MOTOR4_A_OUT -> MOTOR2_CTRL1
- J2 pad 30: MOTOR1_CTRL2 -> MOTOR3_B_OUT
- J2 pad 31: MOTOR1_B_OUT -> MOTOR1_A_OUT
- J2 pad 32: MOTOR1_A_OUT -> MOTOR1_B_OUT
- J2 pad 4: MOTOR2_CTRL1 -> MOTOR4_A_OUT
- J2 pad 5: MOTOR4_B_OUT -> MOTOR2_CTRL2
- J2 pad 6: MOTOR2_CTRL2 -> MOTOR4_B_OUT
- J2 pad 7: CTRL_EXT_LOAD2 -> MOTOR4_CTRL1
- J2 pad 8: MOTOR4_CTRL1 -> CTRL_EXT_LOAD2
- J2 pad 9: unconnected-(J2-Pin_9-Pad9) -> MOTOR4_CTRL2
- JP4 pad 2: BATTERY_POWER -> BATTERY_LOAD
- R12 pad 1: 3V3_OUT -> Net-(JP4-A)
- R31 pad 1: Net-(U7-AISEN) -> Net-(U7-BISEN)
- R33 pad 1: Net-(U4-AISEN) -> Net-(U7-AISEN)
- SW2 pad 1: BATTERY -> CHARGE_BATTERY
- SW2 pad 2: BATTERY_POWER -> BATTERY
- SW2 pad 3: GND -> BATTERY_POWER
- TP11 pad 1: 3V3_OUT -> Net-(JP4-A)
- TP8 pad 1: BATTERY -> CHARGE_BATTERY
- U4 pad 10: MOTOR2_CTRL2 -> MOTOR4_CTRL2
- U4 pad 15: MOTOR1_CTRL2 -> MOTOR2_CTRL2
- U4 pad 16: MOTOR1_CTRL1 -> MOTOR2_CTRL1
- U4 pad 2: MOTOR1_A_OUT -> MOTOR2_A_OUT
- U4 pad 4: MOTOR1_B_OUT -> MOTOR2_B_OUT
- U4 pad 5: MOTOR2_B_OUT -> MOTOR4_B_OUT
- U4 pad 6: Net-(U4-AISEN) -> Net-(U4-BISEN)
- U4 pad 7: MOTOR2_A_OUT -> MOTOR4_A_OUT
- U4 pad 9: MOTOR2_CTRL1 -> MOTOR4_CTRL1
- U5 pad 5: BATTERY -> CHARGE_BATTERY
- U6 pad 1: Net-(U6-L1) -> Net-(U6-EN)
- U6 pad 10: Net-(U6-L2) -> BATTERY_LOAD
- U6 pad 2: BATTERY_LOAD -> GND
- U6 pad 3: /Damola's Sheet/CONN1 -> Net-(U6-FB)
- U6 pad 4: /Damola's Sheet/CONN1 -> 3V3_OUT
- U6 pad 5: Net-(U6-PG) -> (no net)
- U6 pad 6: /Damola's Sheet/CONN1 -> Net-(U6-L2)
- U6 pad 7: GND -> (no net)
- U6 pad 8: Net-(U6-FB) -> Net-(U6-L1)
- U6 pad 9: 3V3_OUT -> (no net)
- U7 pad 10: MOTOR4_CTRL2 -> MOTOR3_CTRL2
- U7 pad 15: MOTOR3_CTRL2 -> MOTOR1_CTRL2
- U7 pad 16: MOTOR3_CTRL1 -> MOTOR1_CTRL1
- U7 pad 2: MOTOR3_A_OUT -> MOTOR1_A_OUT
- U7 pad 4: MOTOR3_B_OUT -> MOTOR1_B_OUT
- U7 pad 5: MOTOR4_B_OUT -> MOTOR3_B_OUT
- U7 pad 6: Net-(U7-AISEN) -> Net-(U7-BISEN)
- U7 pad 7: MOTOR4_A_OUT -> MOTOR3_A_OUT
- U7 pad 9: MOTOR4_CTRL1 -> MOTOR3_CTRL1
- U8 pad 1: Net-(U8-L1) -> Net-(U8-EN)
- U8 pad 10: Net-(U8-L2) -> BATTERY_LOAD
- U8 pad 2: BATTERY_LOAD -> GND
- U8 pad 3: /Damola's Sheet/CONN2 -> Net-(U8-FB)
- U8 pad 4: /Damola's Sheet/CONN2 -> 5V_OUT
- U8 pad 5: Net-(U8-PG) -> (no net)
- U8 pad 6: /Damola's Sheet/CONN2 -> Net-(U8-L2)
- U8 pad 7: GND -> (no net)
- U8 pad 8: Net-(U8-FB) -> Net-(U8-L1)
- U8 pad 9: 5V_OUT -> (no net)
Routing:
- net GND: track 0.00 -> 165.4 mm, vias 0 -> 11
- net BATTERY_LOAD: track 0.00 -> 119.1 mm, vias 0 -> 2
- net 3V3_OUT: track 0.00 -> 117.9 mm, vias 0 -> 4
- net HV: track 0.00 -> 84.1 mm, vias 0 -> 1
- net FAST_CHARGE_CTRL: track 0.00 -> 73.5 mm
- net 5V_OUT: track 0.00 -> 70.3 mm, vias 0 -> 4
- net BATTERY: track 0.00 -> 59.4 mm, vias 0 -> 1
- net /5V: track 0.00 -> 58.0 mm
- net VBUS: track 0.00 -> 49.4 mm
- net MOTOR4_CTRL2: track 0.00 -> 30.4 mm
- net BATTERY_POWER: track 0.00 -> 28.2 mm
- net MOTOR4_CTRL1: track 0.00 -> 27.1 mm
- net Net-(U5-CE): track 0.00 -> 25.9 mm, vias 0 -> 2
- net MOTOR1_CTRL1: track 0.00 -> 25.8 mm, vias 0 -> 1
- net I2C1_SDA: track 0.00 -> 24.6 mm
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- added copper zone on B.Cu, net GND
Other:
- board outline added: 46.5 x 78.5 mm
- board text added: "Micromouse Power Board {dblquote}Great mice are not made by impulse, but by a series of micro decisions brought together.{dblquote} - Mousy Ann Evans"
- board text removed: "JLCJLCJLCJLC"
