File: kicad/shaun-proj/damola.kicad_sch (KiCad schematic)
At the start: 30 parts, among them U4 DRV8833PWPR, U6 TPS63020DSJR, U7 DRV8833PWPR, U8 TPS63020DSJR

Commit message: da board
Parts:
- added R28, R35: 100m, Resistor_SMD:R_1206_3216Metric_Pad1.30x1.75mm_HandSolder, symbol Device:R
- added R29, R36: 1, Resistor_SMD:R_0805_2012Metric_Pad1.20x1.40mm_HandSolder, symbol Device:R
- L4, L5, L6: footprint Inductor_SMD:L_Murata_DFE201610P -> Inductor_SMD:L_1008_2520Metric_Pad1.43x2.20mm_HandSolder
- R34: symbol Device:R_Small_US -> Device:R
- U4, U7: footprint Package_SO:HTSSOP-16-1EP_4.4x5mm_P0.65mm_EP3x3mm -> Package_SO:HTSSOP-16-1EP_4.4x5mm_P0.65mm_EP3.4x5mm_Mask2.46x2.31mm_ThermalVias
- U6, U8: footprint Package_SON:Texas_S-PWSON-N10_ThermalVias -> MyLibrary:DAMOLA_VSON-14-1EP_3.4x4.4mm_P0.5mm_EP1.6x4.2mm; symbol Regulator_Switching:TPS63060 -> CustomSymbols:TPS63020
Connections:
- net 3V3_OUT: now also U6.4 (VOUT); no longer U6.9 (VOUT)
- net 5V_OUT: now also U8.4 (VOUT); no longer U8.9 (VOUT)
- net BATTERY_LOAD: now also U6.10 (VIN), U8.10 (VIN); no longer U6.2 (VIN), U8.2 (VIN)
- net GND: now also U6.15 (PGND), U6.2 (GND), U8.15 (PGND), U8.2 (GND), R28.2, R29.2, R36.2; no longer U6.7 (GND), U8.7 (GND)
- net MOTOR1_A_OUT: now also U7.2 (AOUT1); no longer U4.2 (AOUT1)
- net MOTOR1_B_OUT: now also U7.4 (AOUT2); no longer U4.4 (AOUT2)
- net MOTOR1_CTRL1: now also U7.16 (AIN1); no longer U4.16 (AIN1)
- net MOTOR1_CTRL2: now also U7.15 (AIN2); no longer U4.15 (AIN2)
- net MOTOR2_A_OUT: now also U4.2 (AOUT1); no longer U4.7 (BOUT1)
- net MOTOR2_B_OUT: now also U4.4 (AOUT2); no longer U4.5 (BOUT2)
- net MOTOR2_CTRL1: now also U4.16 (AIN1); no longer U4.9 (BIN1)
- net MOTOR2_CTRL2: now also U4.15 (AIN2); no longer U4.10 (BIN2)
- net MOTOR3_A_OUT: now also U7.7 (BOUT1); no longer U7.2 (AOUT1)
- net MOTOR3_B_OUT: now also U7.5 (BOUT2); no longer U7.4 (AOUT2)
- net MOTOR3_CTRL1: now also U7.9 (BIN1); no longer U7.16 (AIN1)
- net MOTOR3_CTRL2: now also U7.10 (BIN2); no longer U7.15 (AIN2)
- net MOTOR4_A_OUT: now also U4.7 (BOUT1); no longer U7.7 (BOUT1)
- net MOTOR4_B_OUT: now also U4.5 (BOUT2); no longer U7.5 (BOUT2)
- net MOTOR4_CTRL1: now also U4.9 (BIN1); no longer U7.9 (BIN1)
- net MOTOR4_CTRL2: now also U4.10 (BIN2); no longer U7.10 (BIN2)
- net at L5.1: now also U6.6 (L2); no longer U6.10 (L2)
- net at U6.1 (VINA): now also C14.1, U6.12 (EN), U6.13 (PS/SYNC); no longer L4.2
- net at R31.1, U7.6 (BISEN): no longer U7.3 (AISEN)
- net at R32.1, U4.3 (AISEN): now also R29.1; no longer R33.1, U4.6 (BISEN)
- net at R23.2, R24.1: now also U6.3 (FB); no longer U6.8 (FB)
- net at R27.2, R30.1: now also U8.3 (FB); no longer U8.8 (FB)
- net at R25.2: now also U6.14 (PG); no longer U6.5 (PG)
- net at L6.1: now also U8.6 (L2); no longer U8.10 (L2)
- net at L6.2: now also U8.8 (L1); no longer U8.1 (L1)
- net at R34.2: now also U8.14 (PG); no longer U8.5 (PG)
- removed net CONN1: C14.1, U6.3 (EN), U6.4 (PS/SYNC), U6.6 (VAUX)
- removed net CONN2: C22.1, U8.3 (EN), U8.4 (PS/SYNC), U8.6 (VAUX)
- new net: R33.1, R36.1, U7.3 (AISEN)
- new net: L4.2, U6.8 (L1)
- new net: R28.1, R35.2
- new net: R35.1, U4.6 (BISEN)
- new net: C22.1, U8.1 (VINA), U8.12 (EN), U8.13 (PS/SYNC)
Other:
- note added: "MOTOR1 and MOTOR2 need to operate at 200mA, so we'll current-limit at 250mA MOROR3 and MOTOR4 need to operate at 500mA, so we'll current-limit to 600mA We've only got 1ohm and 0.1ohm resistors to work with without incurring, extended feed, so we'll have to settle for 400mA and 1A limit respectively."
- note removed: "Was 450m"
- moved on the sheet: C13, C14, C15, C16, C17, C18, C2, C22, C4, C6, C8, R23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

Commit message: schema improvements, cleanup
Parts:
- added Q10, Q9: AO3401A, Package_TO_SOT_SMD:SOT-23, symbol Transistor_FET:AO3401A
- added Q7, Q8: AO3400A, Package_TO_SOT_SMD:SOT-23, symbol Transistor_FET:AO3400A
- added R37, R38: 10k, Resistor_SMD:R_0603_1608Metric_Pad0.98x0.95mm_HandSolder, symbol Device:R
- added R39, R40: 1M, Resistor_SMD:R_0603_1608Metric_Pad0.98x0.95mm_HandSolder, symbol Device:R
- added SW3: SW_SPDT, MyLibrary:SS-12D11G3R, symbol Switch:SW_SPDT
Connections:
- net 5V_OUT: now also Q10.2 (S), Q9.2 (S), R39.1, R40.1
- net GND: now also Q7.2 (S), Q8.2 (S)
- new net: Q7.1 (G), R37.2
- new net: Q7.3 (D), Q9.1 (G), R39.2
- new net: Q10.1 (G), Q8.3 (D), R40.2
- new net: Q8.1 (G), R38.2
- new net BATTERY: SW3.2 (B)
- new net BATTERY_POWER: SW3.3 (C)
- new net CHARGE_BATTERY: SW3.1 (A)
- new net CTRL_EXT_LOAD1: R37.1
- new net CTRL_EXT_LOAD2: R38.1
- new net EXT_LOAD1_OUT: Q9.3 (D)
- new net EXT_LOAD2_OUT: Q10.3 (D)
Other:
- note added: "External Load Switches"
- note added: "System Power Switch"
- moved on the sheet: C13, C14, C15, C18, C2, C20, C22, C4, C6, L4, L5, L6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
